File: Iota-XL2G4.kicad_pcb (KiCad board)
At the start: 4 copper layers, 10 x 10 mm, 36 parts, among them J1 u.fl, U1 STM32G071EBY6TR, U2 NCP160, U3 SX1280, U4 2450FM07D0034T, Y1 52M

Commit message: general update
Parts:
- removed the TP9 at (130.0, 59.0)
- removed the TP9 at (125.0, 51.0)
- moved C11 0.12 mm to (122.5, 59.6)
Connections:
- U1 pad A1: Net-(U1-PadA1) -> SWDIO
- U1 pad B1: SWDIO -> Net-(U1-PadB1)
- U1 pad C2: Net-(U1-PadC2) -> MISO
- U1 pad D1: MISO -> Net-(U1-PadD1)
- U1 pad D3: Net-(U1-PadD3) -> NRESET
- U1 pad D4: Net-(U1-PadD4) -> NRESET
Routing:
- net NRESET: track 0.00 -> 13.6 mm, vias 1 -> 2
- net Net-(C13-Pad1): track 0.00 -> 8.09 mm, vias 0 -> 2
- net LED1: track 13.7 -> 16.0 mm
- net Net-(J1-Pad1): track 0.00 -> 1.12 mm
- net +3V3: track 0.25 -> 1.27 mm, vias 3 -> 4
- net Net-(C6-Pad1): track 0.00 -> 0.93 mm
- net Net-(U3-Pad22): track 0.00 -> 0.91 mm
- net UART_TX: track 12.1 -> 12.7 mm
- net GND: track 0.27 -> 0.87 mm, vias 10 -> 11
- net NRST: track 7.49 -> 7.77 mm, vias 1 -> 2

Commit message: general update
Parts:
- added REF**: molex_479480001_2g4-turret, footprints:molex_479480001_2g4-turret, F.Cu at (138.6, 55.8)
- moved TP8 12.8 mm to (128.0, 51.0)
- moved TP6 11.7 mm to (124.0, 51.0)
- moved R4 9.65 mm to (127.0, 52.8), turned to 270 degrees
- moved FID3 8.25 mm to (129.2, 60.2)
- moved TP9 8.00 mm to (122.0, 51.0)
- moved C3 7.91 mm to (124.2, 52.9)
- moved U2 7.00 mm to (125.2, 52.9)
- moved C5 6.42 mm to (126.2, 53.0), turned to 270 degrees
- moved TP7 6.00 mm to (126.0, 51.0)
- moved U1 5.97 mm to (128.6, 54.8)
- moved R1 5.60 mm to (125.5, 58.0)
- moved C12 5.21 mm to (124.7, 60.1), turned to 0 degrees
- moved J1 5.07 mm to (127.9, 58.2), turned to 180 degrees
- moved D1 5.03 mm to (125.0, 59.0), turned to 180 degrees
- moved C10 4.82 mm to (128.6, 52.7), turned to 270 degrees
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Routing:
- net LED1: track 16.0 -> 0.00 mm, vias 2 -> 0
- net NRESET: track 13.6 -> 0.00 mm, vias 2 -> 1
- net UART_TX: track 12.7 -> 0.00 mm, vias 1 -> 0
- net BUSY: track 9.92 -> 0.00 mm, vias 2 -> 1
- net SWDIO: track 9.83 -> 0.00 mm, vias 2 -> 1
- net Net-(C13-Pad1): track 8.09 -> 0.00 mm, vias 2 -> 1
- net NRST: track 7.77 -> 0.21 mm, vias 2 -> 1
- net MISO: track 7.57 -> 0.20 mm
- net UART_RX: track 6.35 -> 0.00 mm
- net SWDCLK_BOOT0: track 5.38 -> 0.30 mm
- net DI: track 4.85 -> 0.00 mm
- net SCK: track 3.03 -> 0.19 mm
- net Net-(U3-Pad6): track 2.58 -> 0.00 mm
- net NSS: track 2.41 -> 0.00 mm, vias 2 -> 1
- net MOSI: track 2.10 -> 0.45 mm
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